Commit message: update(melon_description):update urdf and xacro files

File: melon_ws/src/melon_description/urdf/base_v4.xacro (robot description, xacro)
@@ -66,7 +66,29 @@
       </visual>
       <collision>
-        <origin xyz="0.027 0.025 0.37" rpy="0 0 -1.57"/>
+        <!-- <origin xyz="0.027 0.025 0.37" rpy="0 0 -1.57"/>
         <geometry>
           <mesh filename="package://melon_description/meshes/body_3.stl" scale="0.001 0.001 0.001"/>
+        </geometry> -->
+        <origin xyz="0.008 0.0 0.415" rpy="0 0 0"/>
+        <geometry>
+          <box size="0.8 0.7 0.1"/>
+        </geometry>
+      </collision>
+      <collision>
+        <origin xyz="0.258 0.0 0.615" rpy="0 0 0"/>
+        <geometry>
+          <box size="0.3 0.7 0.3"/>
+        </geometry>
+      </collision>
+      <collision>
+        <origin xyz="-0.14 0.335 0.495" rpy="0 0 0"/>
+        <geometry>
+          <box size="0.5 0.03 0.06"/>
+        </geometry>
+      </collision>
+      <collision>
+        <origin xyz="-0.14 -0.335 0.495" rpy="0 0 0"/>
+        <geometry>
+          <box size="0.5 0.03 0.06"/>
         </geometry>
       </collision>

File: melon_ws/src/melon_description/urdf/melon.urdf (robot description, URDF)
Before this commit: robot Melon, 41 links, 40 joints
Links:
- link base_link: geometry collision box size=0.3 0.7 0.3; collision box size=0.5 0.03 0.06
